Commit message: updates base link name and add virtual joint for ros2_control

File: onrobot_descriptions/urdf/vg_series/vg10/vg10_macro.xacro (robot description, xacro)
@@ -6,5 +6,5 @@
   <xacro:macro name="onrobot_vg10" params="prefix">
     <!-- Base Link -->
-    <link name="${prefix}onrobot_vg10_base_link">
+    <link name="${prefix}onrobot_vg_base_link">
       <inertial>
         <origin xyz="0.0 0.0 0.0" rpy="0 0 0" />
@@ -38,5 +38,5 @@
         <origin xyz="0 0 0" rpy="0 0 0" />
         <geometry>
-          <mesh filename="package://onrobot_descriptions/meshes/vg_series/vg10/visual/suction_pad.stl" />
+          <mesh filename="package://onrobot_descriptions/meshes/vg_series/vg10/visual/suction_cups.stl" />
         </geometry>
         <material name="">
@@ -47,5 +47,5 @@
         <origin xyz="0 0 0" rpy="0 0 0" />
         <geometry>
-          <mesh filename="package://onrobot_descriptions/meshes/vg_series/vg10/collision/suction_pad.stl" />
+          <mesh filename="package://onrobot_descriptions/meshes/vg_series/vg10/collision/suction_cups.stl" />
         </geometry>
       </collision>
@@ -53,6 +53,22 @@
     <joint name="${prefix}_suction_pad_joint" type="fixed">
       <origin xyz="0 0 0.12" rpy="0 0 0" />
-      <parent link="${prefix}onrobot_vg10_base_link" />
+      <parent link="${prefix}onrobot_vg_base_link" />
       <child link="${prefix}suction_pad" />
+    </joint>
+    <!-- Virtual suction regulator link for ros2_control -->
+    <link name="${prefix}suction_regulator">
+      <inertial>
+        <mass value="0.001"/>
+        <inertia ixx="1.0E-09" ixy="0.0" ixz="0.0" iyy="1.0E-09" iyz="0.0" izz="1.0E-09"/>
+      </inertial>
+    </link>
+    <!-- Virtual joint for vacuum control (0-80 kPa) -->
+    <joint name="${prefix}_suction_regulator_joint" type="prismatic">
+      <origin xyz="0 0 0" rpy="0 0 0"/>
+      <parent link="${prefix}onrobot_vg_base_link"/>
+      <child link="${prefix}suction_regulator"/>
+      <axis xyz="0 0 1"/>
+      <limit lower="0.0" upper="80.0" effort="100.0" velocity="0.2"/>
+      <dynamics damping="0.1" friction="0.0"/>
     </joint>
   </xacro:macro>

File: onrobot_descriptions/urdf/vg_series/vgc10/vgc10_macro.xacro (robot description, xacro)
@@ -14,5 +14,5 @@
          BASE LINK
          ═══════════════════════════════════════════════════════════════ -->
-    <link name="${prefix}onrobot_vgc10_base_link">
+    <link name="${prefix}onrobot_vg_base_link">
       <inertial>
         <origin xyz="0.0 0.0 0.0" rpy="0 0 0" />
@@ -65,5 +65,5 @@
       <joint name="${prefix}_suction_joint" type="fixed">
         <origin xyz="0 0 0.094901" rpy="0 0 0" />
-        <parent link="${prefix}onrobot_vgc10_base_link" />
+        <parent link="${prefix}onrobot_vg_base_link" />
         <child link="${prefix}suction" />
       </joint>
@@ -103,23 +103,39 @@
       <joint name="${prefix}_suction_joint1" type="fixed">
         <origin xyz="0.050 -0.050 0.094901" rpy="0 0 0" />
-        <parent link="${prefix}onrobot_vgc10_base_link" />
+        <parent link="${prefix}onrobot_vg_base_link" />
         <child link="${prefix}suction1" />
       </joint>
       <joint name="${prefix}_suction_joint2" type="fixed">
         <origin xyz="0.050 0.050 0.094901" rpy="0 0 0" />
-        <parent link="${prefix}onrobot_vgc10_base_link" />
+        <parent link="${prefix}onrobot_vg_base_link" />
         <child link="${prefix}suction2" />
       </joint>
       <joint name="${prefix}_suction_joint3" type="fixed">
         <origin xyz="-0.050 -0.050 0.094901" rpy="0 0 0" />
-        <parent link="${prefix}onrobot_vgc10_base_link" />
+        <parent link="${prefix}onrobot_vg_base_link" />
         <child link="${prefix}suction3" />
       </joint>
       <joint name="${prefix}_suction_joint4" type="fixed">
         <origin xyz="-0.050 0.050 0.094901" rpy="0 0 0" />
-        <parent link="${prefix}onrobot_vgc10_base_link" />
+        <parent link="${prefix}onrobot_vg_base_link" />
         <child link="${prefix}suction4" />
       </joint>
     </xacro:if>
+    <!-- Virtual suction regulator link for ros2_control -->
+    <link name="${prefix}suction_regulator">
+      <inertial>
+        <mass value="0.001"/>
+        <inertia ixx="1.0E-09" ixy="0.0" ixz="0.0" iyy="1.0E-09" iyz="0.0" izz="1.0E-09"/>
+      </inertial>
+    </link>
+    <!-- Virtual joint for vacuum control (0-80 kPa) -->
+    <joint name="${prefix}_suction_regulator_joint" type="prismatic">
+      <origin xyz="0 0 0" rpy="0 0 0"/>
+      <parent link="${prefix}onrobot_vg_base_link"/>
+      <child link="${prefix}suction_regulator"/>
+      <axis xyz="0 0 1"/>
+      <limit lower="0.0" upper="80.0" effort="100.0" velocity="0.2"/>
+      <dynamics damping="0.1" friction="0.0"/>
+    </joint>
   </xacro:macro>
 </robot>
